File: PCB/kolko_4layer.kicad_sch (KiCad schematic)
At the start: 81 parts, among them IC1 74HC4067PW-Q100J, J1 USB_C_Receptacle_USB2.0_16P, J2 Conn_01x02_Socket, J3 Conn_01x04_Socket, SW1 RST, SW2 BOOT, U1 ESP32-S3-WROOM-1, U2 USBLC6-2SC6, U3 AMS1117-3.3

Commit message: usb reroute
Parts:
- J3: footprint Connector_PinHeader_2.54mm:PinHeader_1x04_P2.54mm_Vertical -> Connector_Molex:Molex_PicoBlade_53047-0410_1x04_P1.25mm_Vertical
Connections:
- net +3.3V: now also J3.1 (Pin_1); no longer J3.4 (Pin_4)
- net GND: now also J3.4 (Pin_4); no longer J3.1 (Pin_1)
- net D_1MCU+: now reaches U1.14 (USB_D+), U2.6 (I/O1)
- no-connect marks 0 -> 2
Changed lines of the file:
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@@
 	(wire
 		(pts
+			(xy 83.82 110.49) (xy 83.82 111.76)
+		)
+		(stroke
+			(width 0)
+			(type default)
+		)
+	)
+	(wire
+		(pts
 			(xy 165.1 180.34) (xy 167.64 180.34)
 		)
@@
 	(wire
 		(pts
-			(xy 77.47 111.76) (xy 85.09 111.76)
+			(xy 83.82 110.49) (xy 85.09 110.49)
 		)
 		(stroke
@@
 	(wire
 		(pts
+			(xy 85.09 119.38) (xy 85.09 121.92)
+		)
+		(stroke
+			(width 0)
+			(type default)
+		)
+	)
+	(wire
+		(pts
 			(xy 181.61 58.42) (xy 186.69 58.42)
 		)
@@
 	(wire
 		(pts
-			(xy 266.7 53.34) (xy 267.97 53.34)
-		)
-		(stroke
-			(width 0)
-			(type default)
-		)
-	)
-	(wire
-		(pts
 			(xy 132.08 102.87) (xy 134.62 102.87)
 		)
@@
 	(wire
 		(pts
-			(xy 85.09 111.76) (xy 85.09 110.49)
-		)
-		(stroke
-			(width 0)
-			(type default)
-		)
-	)
-	(wire
-		(pts
 			(xy 114.3 26.67) (xy 118.11 26.67)
 		)
@@
 	(wire
 		(pts
+			(xy 83.82 111.76) (xy 77.47 111.76)
+		)
+		(stroke
+			(width 0)
+			(type default)
+		)
+	)
+	(wire
+		(pts
 			(xy 165.1 149.86) (xy 167.64 149.86)
 		)
@@
 		)
 	)
+	(no_connect
+		(at 242.57 54.61)
+	)
+	(no_connect
+		(at 242.57 57.15)
+	)
 	(label "D_1MCU+"
-		(at 267.97 53.34 0)
+		(at 266.7 53.34 0)
 		(effects
 			(font
@@
 		)
 	)
-	(label ""
-		(at 266.7 53.34 0)
-		(effects
-			(font
-				(size 1.27 1.27)
-			)
-			(justify left bottom)
-		)
-	)
 	(label "VEXT"
 		(at 114.3 26.67 180)
@@
 	(symbol
 		(lib_id "power:+3.3V")
-		(at 85.09 110.49 270)
+		(at 85.09 121.92 270)
 		(unit 1)
 		(exclude_from_sim no)
@@
 		(fields_autoplaced yes)
 		(property "Reference" "#PWR040"
-			(at 81.28 110.49 0)
+			(at 81.28 121.92 0)
 			(effects
 				(font
@@
 		)
 		(property "Value" "+3.3V"
-			(at 88.9 110.4899 90)
+			(at 88.9 121.9199 90)
 			(effects
 				(font
@@
 		)
 		(property "Footprint" ""
-			(at 85.09 110.49 0)
+			(at 85.09 121.92 0)
 			(effects
 				(font
@@
 		)
 		(property "Datasheet" ""
-			(at 85.09 110.49 0)
+			(at 85.09 121.92 0)
 			(effects
 				(font
@@
 		)
 		(property "Description" "Power symbol creates a global label with name \"+3.3V\""
-			(at 85.09 110.49 0)
+			(at 85.09 121.92 0)
 			(effects
 				(font
@@
 		)
 		(instances
-			(project ""
+			(project "kolko_4layer"
 				(path "/f490b379-6bd6-444b-87af-8b43edc8fb8b"
 					(reference "#PWR040")
@@
 	(symbol
 		(lib_id "power:GND")
-		(at 85.09 119.38 90)
+		(at 85.09 110.49 90)
 		(unit 1)
 		(exclude_from_sim no)
@@
 		(fields_autoplaced yes)
 		(property "Reference" "#PWR020"
-			(at 91.44 119.38 0)
+			(at 91.44 110.49 0)
 			(effects
 				(font
@@
 		)
 		(property "Value" "GND"
-			(at 88.9 119.3799 90)
+			(at 88.9 110.4899 90)
 			(effects
 				(font
@@
 		)
 		(property "Footprint" ""
-			(at 85.09 119.38 0)
+			(at 85.09 110.49 0)
 			(effects
 				(font
@@
 		)
 		(property "Datasheet" ""
-			(at 85.09 119.38 0)
+			(at 85.09 110.49 0)
 			(effects
 				(font
@@
 		)
 		(property "Description" "Power symbol creates a global label with name \"GND\" , ground"
-			(at 85.09 119.38 0)
+			(at 85.09 110.49 0)
 			(effects
 				(font
@@
 		)
 		(instances
-			(project ""
+			(project "kolko_4layer"
 				(path "/f490b379-6bd6-444b-87af-8b43edc8fb8b"
 					(reference "#PWR020")
@@
 			)
 		)
-		(property "Footprint" "Connector_PinHeader_2.54mm:PinHeader_1x04_P2.54mm_Vertical"
+		(property "Footprint" "Connector_Molex:Molex_PicoBlade_53047-0410_1x04_P1.25mm_Vertical"
 			(at 72.39 116.84 0)
 			(effects

Commit message: kosmetyczne zmiany
Parts:
- D1, D2: footprint LED_SMD:LED_0805_2012Metric -> Diode_SMD:D_SMB
- IC1: footprint muxy2:SOP65P640X110-24N -> Package_SO:TSSOP-24_4.4x7.8mm_P0.65mm
- U3: value AMS1117-3.3 -> TLV76133DCYR
Changed lines of the file:
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@@
 		(color 0 0 0 0)
 	)
+	(no_connect
+		(at 242.57 54.61)
+	)
+	(no_connect
+		(at 242.57 57.15)
+	)
 	(wire
 		(pts
@@
 		)
 	)
-	(no_connect
-		(at 242.57 54.61)
-	)
-	(no_connect
-		(at 242.57 57.15)
-	)
 	(label "D_1MCU+"
 		(at 266.7 53.34 0)
@@
 			)
 		)
-		(property "Footprint" "muxy2:SOP65P640X110-24N"
+		(property "Footprint" "Package_SO:TSSOP-24_4.4x7.8mm_P0.65mm"
 			(at 49.53 257.48 0)
 			(effects
@@
 			)
 		)
-		(property "Value" "AMS1117-3.3"
+		(property "Value" "TLV76133DCYR"
 			(at 127 48.26 0)
 			(effects
@@
 			)
 		)
-		(property "Footprint" "LED_SMD:LED_0805_2012Metric"
+		(property "Footprint" "Diode_SMD:D_SMB"
 			(at 182.88 25.4 0)
 			(effects
@@
 			)
 		)
-		(property "Footprint" "LED_SMD:LED_0805_2012Metric"
+		(property "Footprint" "Diode_SMD:D_SMB"
 			(at 182.88 34.29 0)
 			(effects
